File: miniamp_board/miniamp_board.kicad_pcb (KiCad board)
At the start: 2 copper layers, 55.2 x 31.1 mm, 29 parts, among them J1 Conn_01x03, SW1 ON_OFF, U1 LM4871M

Commit message: wip
Parts:
- J1: value Conn_01x03 -> AUDIO_IN
- SW1: value ON_OFF -> MAIN
- moved SW_1 102.7 mm to (116.2, 102.9)
- moved SW_2 98.7 mm to (116.2, 99.7)
- moved BT1 96.8 mm to (128.3, 95.2)
- moved C3 96.8 mm to (146.1, 101.6)
- moved C4 96.8 mm to (149.9, 104.1)
- moved J1 96.8 mm to (148.6, 95.2)
- moved LS1 96.8 mm to (157.4, 95.2)
- moved R1 96.8 mm to (142.2, 111.1)
- moved R3 96.8 mm to (130.8, 111.1)
- moved R4 96.8 mm to (134.6, 111.1)
- moved R5 96.8 mm to (138.4, 111.1)
- moved REF** 96.8 mm to (118.7, 98.4)
- moved REF** 96.8 mm to (165.7, 110.5)
- moved REF** 96.8 mm to (165.7, 87.0)
- moved C1 96.8 mm to (125.1, 106.0)
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Connections:
- C1 pad 1: Net-(BT1-Pad1) -> +BATT
- C2 pad 1: Net-(BT1-Pad1) -> +BATT
- SW1 pad 1: +BATT -> Net-(BT1-Pad1)
- SW1 pad 2: Net-(BT1-Pad1) -> +BATT
Routing:
- net +BATT: track 65.8 -> 73.4 mm
- net Net-(BT1-Pad1): track 32.6 -> 37.2 mm
- net GND: track 2.35 -> 6.90 mm, vias 9 -> 20
