File: miniamp_board/miniamp_board.sch (KiCad schematic (older format))
At the start: 15 parts, among them J1 Conn_01x03, SW1 ON_OFF, U1 LM4871M

Commit message: wip
Parts:
- J1: value Conn_01x03 -> AUDIO_IN
- SW1: value ON_OFF -> MAIN
Connections:
- net +BATT: now also SW1.2 (B); no longer SW1.1 (A)
- net at BT1.1 (+): now also SW1.1 (A); no longer SW1.2 (B)
Other:
- moved on the sheet: C1, C2
Changed lines of the file:
@@
 L power:+BATT #PWR01
 U 1 1 5F3B53CF
-P 1550 2900
-F 0 "#PWR01" H 1550 2750 50  0001 C CNN
-F 1 "+BATT" H 1565 3073 50  0000 C CNN
-F 2 "" H 1550 2900 50  0001 C CNN
-F 3 "" H 1550 2900 50  0001 C CNN
-	1    1550 2900
+P 2750 2900
+F 0 "#PWR01" H 2750 2750 50  0001 C CNN
+F 1 "+BATT" H 2765 3073 50  0000 C CNN
+F 2 "" H 2750 2900 50  0001 C CNN
+F 3 "" H 2750 2900 50  0001 C CNN
+	1    2750 2900
 	1    0    0    -1
 $EndComp
@@
 AUDIO_INPUT
 Wire Wire Line
-	1550 3200 1550 3050
-Wire Wire Line
 	1550 4200 1550 4500
 $Comp
@@
 P 8000 3600
 F 0 "J1" H 7918 3275 50  0000 C CNN
-F 1 "Conn_01x03" H 7918 3366 50  0000 C CNN
+F 1 "AUDIO_IN" H 7918 3366 50  0000 C CNN
 F 2 "Connector_JST:JST_XH_S3B-XH-A_1x03_P2.50mm_Horizontal" H 8000 3600 50  0001 C CNN
 F 3 "~" H 8000 3600 50  0001 C CNN
@@
 	-1   0    0    1
 $EndComp
-$Comp
-L Switch:SW_SPST SW1
-U 1 1 5F3E7791
-P 1550 3400
-F 0 "SW1" V 1504 3312 50  0000 R CNN
-F 1 "ON_OFF" V 1595 3312 50  0000 R CNN
-F 2 "Connector_JST:JST_XH_S2B-XH-A_1x02_P2.50mm_Horizontal" H 1550 3400 50  0001 C CNN
-F 3 "~" H 1550 3400 50  0001 C CNN
-	1    1550 3400
-	0    -1   1    0
-$EndComp
-$Comp
-L power:+BATT #PWR06
-U 1 1 5F489421
-P 5350 2900
-F 0 "#PWR06" H 5350 2750 50  0001 C CNN
-F 1 "+BATT" H 5365 3073 50  0000 C CNN
-F 2 "" H 5350 2900 50  0001 C CNN
-F 3 "" H 5350 2900 50  0001 C CNN
-	1    5350 2900
-	1    0    0    -1
-$EndComp
-Connection ~ 5350 2900
 Wire Notes Line
 	3300 4800 7500 4800
@@
 L Device:CP C1
 U 1 1 5F4CE2AC
-P 2200 3400
-F 0 "C1" H 2318 3446 50  0000 L CNN
-F 1 "100uF" H 2318 3355 50  0000 L CNN
-F 2 "Capacitor_THT:CP_Radial_D6.3mm_P2.50mm" H 2238 3250 50  0001 C CNN
-F 3 "~" H 2200 3400 50  0001 C CNN
-	1    2200 3400
+P 2200 4000
+F 0 "C1" H 2318 4046 50  0000 L CNN
+F 1 "100uF" H 2318 3955 50  0000 L CNN
+F 2 "Capacitor_THT:CP_Radial_D6.3mm_P2.50mm" H 2238 3850 50  0001 C CNN
+F 3 "~" H 2200 4000 50  0001 C CNN
+	1    2200 4000
 	1    0    0    -1
 $EndComp
@@
 L Device:C C2
 U 1 1 5F4CF21E
-P 2750 3400
-F 0 "C2" H 2865 3446 50  0000 L CNN
-F 1 "0.1u" H 2865 3355 50  0000 L CNN
-F 2 "Capacitor_THT:C_Disc_D5.0mm_W2.5mm_P2.50mm" H 2788 3250 50  0001 C CNN
-F 3 "~" H 2750 3400 50  0001 C CNN
-	1    2750 3400
-	1    0    0    -1
-$EndComp
-Wire Wire Line
-	1550 3050 2200 3050
-Wire Wire Line
-	2200 3050 2200 3250
-Wire Wire Line
-	2750 3050 2750 3250
+P 2750 4000
+F 0 "C2" H 2865 4046 50  0000 L CNN
+F 1 "0.1u" H 2865 3955 50  0000 L CNN
+F 2 "Capacitor_THT:C_Disc_D5.0mm_W2.5mm_P2.50mm" H 2788 3850 50  0001 C CNN
+F 3 "~" H 2750 4000 50  0001 C CNN
+	1    2750 4000
+	1    0    0    -1
+$EndComp
 $Comp
 L power:GND #PWR03
@@
 	3150 4800 1350 4800
 Wire Wire Line
-	2200 3050 2750 3050
-Connection ~ 2200 3050
-Connection ~ 1550 3050
-Wire Wire Line
-	1550 3050 1550 2900
-Wire Wire Line
-	1550 3600 1550 3800
-Wire Wire Line
-	2200 3550 2200 4500
-Wire Wire Line
-	2750 3550 2750 4500
+	2200 3400 2750 3400
+$Comp
+L Switch:SW_SPST SW1
+U 1 1 5F3D47E1
+P 1850 3400
+F 0 "SW1" H 1850 3635 50  0000 C CNN
+F 1 "MAIN" H 1850 3544 50  0000 C CNN
+F 2 "Connector_JST:JST_XH_S2B-XH-A_1x02_P2.50mm_Horizontal" H 1850 3400 50  0001 C CNN
+F 3 "~" H 1850 3400 50  0001 C CNN
+	1    1850 3400
+	1    0    0    -1
+$EndComp
+Wire Wire Line
+	1550 3800 1550 3400
+Wire Wire Line
+	2200 3400 2200 3850
+Wire Wire Line
+	2750 3400 2750 3850
+Wire Wire Line
+	2200 4500 2200 4150
+Wire Wire Line
+	2750 4150 2750 4500
+Wire Wire Line
+	2750 2900 2750 3400
+Connection ~ 2750 3400
+$Comp
+L power:+BATT #PWR0101
+U 1 1 5F3E2F0E
+P 5350 2900
+F 0 "#PWR0101" H 5350 2750 50  0001 C CNN
+F 1 "+BATT" H 5365 3073 50  0000 C CNN
+F 2 "" H 5350 2900 50  0001 C CNN
+F 3 "" H 5350 2900 50  0001 C CNN
+	1    5350 2900
+	1    0    0    -1
+$EndComp
+Connection ~ 5350 2900
+Wire Wire Line
+	2050 3400 2200 3400
+Connection ~ 2200 3400
+Wire Wire Line
+	1550 3400 1650 3400
 $EndSCHEMATC
